Commit message: Added wheels to the robot with continous joint

File: urdf/my_robot.urdf (robot description, URDF)
Before this commit: robot my_bot, 2 links, 1 joints
Links:
- removed link lidar_link
- added link left_wheel; visual cylinder length=0.02 radius=0.05
- added link right_wheel; visual cylinder length=0.02 radius=0.05
- link base_link: mass None -> 1.0; geometry collision box size=0.4 0.3 0.1; visual box size=0.4 0.3 0.1
Joints:
- removed joint lidar_joint
- added joint left_wheel_joint: type fixed, parent base_link, child left_wheel, origin xyz=0 -0.15 -0.05 rpy=0 0 0
- added joint right_wheel_joint: type fixed, parent base_link, child right_wheel, origin xyz=0 0.15 -0.05 rpy=0 0 0
